Commit message: add dummy inertias to motoman_hc10dt_support urdfs
These tags are needed in order for the robot to be used in Gazebo.

File: motoman_hc10_support/urdf/hc10_macro.xacro (robot description, xacro)
@@ -19,4 +19,8 @@
         </geometry>
       </collision>
+      <inertial>
+        <mass value="0.1" />
+        <inertia ixx="0.03" iyy="0.03" izz="0.03" ixy="0.0" ixz="0.0" iyz="0.0" />
+      </inertial>
     </link>
     <link name="${prefix}link_1_s">
@@ -32,4 +36,8 @@
         </geometry>
       </collision>
+      <inertial>
+        <mass value="0.1" />
+        <inertia ixx="0.03" iyy="0.03" izz="0.03" ixy="0.0" ixz="0.0" iyz="0.0" />
+      </inertial>
     </link>
     <link name="${prefix}link_2_l">
@@ -45,4 +53,8 @@
         </geometry>
       </collision>
+      <inertial>
+        <mass value="0.1" />
+        <inertia ixx="0.03" iyy="0.03" izz="0.03" ixy="0.0" ixz="0.0" iyz="0.0" />
+      </inertial>
     </link>
     <link name="${prefix}link_3_u">
@@ -58,4 +70,8 @@
         </geometry>
       </collision>
+      <inertial>
+        <mass value="0.1" />
+        <inertia ixx="0.03" iyy="0.03" izz="0.03" ixy="0.0" ixz="0.0" iyz="0.0" />
+      </inertial>
     </link>
     <link name="${prefix}link_4_r">
@@ -71,4 +87,8 @@
         </geometry>
       </collision>
+      <inertial>
+        <mass value="0.1" />
+        <inertia ixx="0.03" iyy="0.03" izz="0.03" ixy="0.0" ixz="0.0" iyz="0.0" />
+      </inertial>
     </link>
     <link name="${prefix}link_5_b">
@@ -84,4 +104,8 @@
         </geometry>
       </collision>
+      <inertial>
+        <mass value="0.1" />
+        <inertia ixx="0.03" iyy="0.03" izz="0.03" ixy="0.0" ixz="0.0" iyz="0.0" />
+      </inertial>
     </link>
     <link name="${prefix}link_6_t">
@@ -97,4 +121,8 @@
         </geometry>
       </collision>
+      <inertial>
+        <mass value="0.1" />
+        <inertia ixx="0.03" iyy="0.03" izz="0.03" ixy="0.0" ixz="0.0" iyz="0.0" />
+      </inertial>
     </link>
     <link name="${prefix}tool0"/>

File: motoman_hc10_support/urdf/hc10dt_macro.xacro (robot description, xacro)
@@ -22,4 +22,8 @@
         </geometry>
       </collision>
+      <inertial>
+        <mass value="0.1" />
+        <inertia ixx="0.03" iyy="0.03" izz="0.03" ixy="0.0" ixz="0.0" iyz="0.0" />
+      </inertial>
     </link>
     <link name="${prefix}link_1_s">
@@ -35,4 +39,8 @@
         </geometry>
       </collision>
+      <inertial>
+        <mass value="0.1" />
+        <inertia ixx="0.03" iyy="0.03" izz="0.03" ixy="0.0" ixz="0.0" iyz="0.0" />
+      </inertial>
     </link>
     <link name="${prefix}link_2_l">
@@ -48,4 +56,8 @@
         </geometry>
       </collision>
+      <inertial>
+        <mass value="0.1" />
+        <inertia ixx="0.03" iyy="0.03" izz="0.03" ixy="0.0" ixz="0.0" iyz="0.0" />
+      </inertial>
     </link>
     <link name="${prefix}link_3_u">
@@ -61,4 +73,8 @@
         </geometry>
       </collision>
+      <inertial>
+        <mass value="0.1" />
+        <inertia ixx="0.03" iyy="0.03" izz="0.03" ixy="0.0" ixz="0.0" iyz="0.0" />
+      </inertial>
     </link>
     <link name="${prefix}link_4_r">
@@ -74,4 +90,8 @@
         </geometry>
       </collision>
+      <inertial>
+        <mass value="0.1" />
+        <inertia ixx="0.03" iyy="0.03" izz="0.03" ixy="0.0" ixz="0.0" iyz="0.0" />
+      </inertial>
     </link>
     <link name="${prefix}link_5_b">
@@ -87,4 +107,8 @@
         </geometry>
       </collision>
+      <inertial>
+        <mass value="0.1" />
+        <inertia ixx="0.03" iyy="0.03" izz="0.03" ixy="0.0" ixz="0.0" iyz="0.0" />
+      </inertial>
     </link>
     <link name="${prefix}link_6_t">
@@ -100,4 +124,8 @@
        </geometry>
       </collision>
+      <inertial>
+        <mass value="0.1" />
+        <inertia ixx="0.03" iyy="0.03" izz="0.03" ixy="0.0" ixz="0.0" iyz="0.0" />
+      </inertial>
     </link>
     <link name="${prefix}tool0"/>
